Commit message: Updated to the 0.7.3 release.

File: WSU-Portable-Generator/source/partial_env_generator/envs/cartpolepp/models/ground_cart.urdf (robot description, URDF)
Before this commit: robot ground, 3 links, 2 joints
Links:
- link cart: mass 1 -> 1.0
- link ground: geometry collision box size=0.01 0.01 0.01; visual box size=0.1 0.1 0.3
- link pole: mass 1 -> 0.1
Joints:
- joint ground_to_cart: origin xyz=0.0 0.0 0.0 -> xyz=0.0 0.0 0.0 rpy=0.0 0.0 0.0

Commit message: removed debugging code breaking behaviour

File: WSU-Portable-Generator/source/partial_env_generator/envs/cartpolepp/models/ground_cart.urdf (robot description, URDF)
Before this commit: robot ground, 3 links, 2 joints
Links:
- link ground: geometry collision box size=0.01 0.01 0.01; visual box size=0.01 0.01 0.01
